File: PCB/Vehicle Power Switch.kicad_pcb (KiCad board)
At the start: 2 copper layers, 76.5 x 85 mm, 47 parts, among them J6 STX-3790-5N, J7 Debug Hdr, J8 AVR-UPDI-6, Q1 MMBT2222A, Q2 MMBT2222A, Q3 BSS84, U1 MCP1703Ax-250xxTT, U2 LIS2HH12, U3 ATtiny404-SS

Commit message: Fixes to PCB v2 and working on firmware.
Connections:
- U2 pad 5: unconnected-(U2-RES-Pad5) -> GND

Commit message: All functionality is working on the prototype. Firmware is still rough.
Parts:
- added C2: 10nF, Capacitor_SMD:C_0805_2012Metric, F.Cu at (94.0, 59.5)
- added C3: 22uF, Capacitor_SMD:C_0805_2012Metric, F.Cu at (102.0, 59.5)
- C1: value .1uF -> 22uF
- C10: renamed from C9; value .1uF -> 10nF
- C4: renamed from C3; value 10uF -> 10nF; footprint Capacitor_SMD:CP_Elec_4x5.3 -> Capacitor_SMD:C_0805_2012Metric
- C5: renamed from C4; value .1uF -> 10nF
- C6: renamed from C5; value .1uF -> 10nF
- C7: value .1uF -> 10nF
- C8: renamed from C6; value .1uF -> 10nF
- C9: renamed from C8; value .1uF -> 10nF
- D1, D2, D3, D5: value MRA4007T3G -> 1N4007FL; footprint Diode_SMD:D_SMA -> Diode_SMD:D_SOD-123
- D4: footprint LED_SMD:LED_1206_3216Metric -> LED_SMD:LED_0805_2012Metric
- moved C6 51.6 mm to (110.0, 107.6), turned to 90 degrees
- moved J8 32.9 mm to (77.1, 130.2)
- moved R5 31.5 mm to (94.0, 124.5)
- moved C5 29.1 mm to (104.0, 124.5), turned to 90 degrees
- moved D4 25.8 mm to (97.0, 125.1)
- moved R9 24.8 mm to (113.0, 84.4), turned to -90 degrees
- moved R3 23.5 mm to (107.0, 124.5)
- moved R2 23.2 mm to (110.0, 124.5)
- moved J7 22.5 mm to (97.4, 130.3), turned to -90 degrees
- moved U2 22.1 mm to (106.7, 129.8)
- moved D3 21.1 mm to (91.0, 125.2)
- moved R10 19.1 mm to (116.0, 90.4)
- moved D2 18.8 mm to (92.7, 63.7)
- moved Q3 18.4 mm to (112.7, 79.3)
- moved Q2 18.3 mm to (107.3, 79.3)
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- renumbered U4 to K1
Connections:
- R7 pad 1: Net-(U3-PA3) -> GND
- R7 pad 3: GND -> Net-(U3-PA3)
- U2 pad 3: unconnected-(U2-SA0/SDO-Pad3) -> +3V3
Routing:
- net GND: track 1.50 -> 128.4 mm, vias 59 -> 112
- net /1: track 69.4 -> 137.8 mm
- net /2: track 66.8 -> 129.6 mm
- net Net-(D2-A): track 31.8 -> 54.2 mm
- net Net-(J8-DATA): track 30.6 -> 52.1 mm
- net Net-(J7-Pin_2): track 6.69 -> 23.4 mm
- net Net-(U3-PA7): track 30.1 -> 16.1 mm, vias 0 -> 2
- net /PB1: track 9.89 -> 23.1 mm
- net Net-(J7-Pin_1): track 6.84 -> 19.2 mm
- net /In: track 22.6 -> 31.1 mm
- net Net-(Q3-D): track 6.03 -> 12.8 mm
- net Net-(D4-A): track 15.5 -> 21.7 mm
- net Net-(U3-PA5): track 37.8 -> 32.2 mm
- net +3V3: track 114.9 -> 120.3 mm, vias 6 -> 4
- net +BATT: track 139.1 -> 134.0 mm, vias 2 -> 3
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Other:
- board size 76.5 x 85 mm -> 62 x 83 mm
- board text added: "Debug"
- board text added: "INPUT"
- board text added: "OUTPUTS"
- board text added: "On-Off-Auto Sw"
- board text added: "Threshold"
- board text added: "UPDI"
- board text added: "Vehicle Power Switch v2.1.1 Zack Clobes, W0ZC Custom Digital Services, LLC"
- board text removed: "Vehicle Power Switch v2.0 Zack Clobes, W0ZC Custom Digital Services, LLC"

Commit message: Release candidate for firmware.
Parts:
- moved D4 0.70 mm to (97.0, 124.4)
Connections:
- J7 pad 1: Net-(J7-Pin_1) -> unconnected-(J7-Pin_1-Pad1)
- U3 pad 7: Net-(J7-Pin_1) -> unconnected-(U3-PB2-Pad7)
Routing:
- net Net-(J7-Pin_1): track 19.2 -> 0.00 mm
- net Net-(D4-A): track 21.7 -> 20.0 mm
- net Net-(J7-Pin_2): track 23.4 -> 22.5 mm
- net GND: vias 112 -> 113
Other:
- board text added: "MAXIMUM 30 AMP TOTAL CONSUMPTION!!!"
- board text added: "Vehicle Power Switch v2.1.2 Zack Clobes, W0ZC Custom Digital Services, LLC"
- board text removed: "Vehicle Power Switch v2.1.1 Zack Clobes, W0ZC Custom Digital Services, LLC"
Changed lines of the file:
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@@
 			(pdf_back_fp_property_popups yes)
 			(pdf_metadata yes)
-			(pdf_single_document no)
+			(pdf_single_document yes)
 			(dxfpolygonmode yes)
 			(dxfimperialunits yes)
@@
 			(crossoutdnponfab yes)
 			(subtractmaskfromsilk no)
-			(outputformat 1)
+			(outputformat 4)
 			(mirror no)
 			(drillshape 0)
@@
 	(net 10 "Net-(D4-K)")
 	(net 11 "Net-(J7-Pin_2)")
-	(net 12 "Net-(J7-Pin_1)")
+	(net 12 "unconnected-(J7-Pin_1-Pad1)")
 	(net 13 "unconnected-(J8-NC-Pad5)")
 	(net 14 "unconnected-(J8-NC-Pad3)")
@@
 	(net 29 "/PB0")
 	(net 30 "/PB1")
+	(net 31 "unconnected-(U3-PB2-Pad7)")
 	(footprint "Package_TO_SOT_SMD:SOT-23"
 		(layer "F.Cu")
@@
 			(layers "F.Cu" "F.Mask" "F.Paste")
 			(roundrect_rratio 0.25)
-			(net 12 "Net-(J7-Pin_1)")
+			(net 31 "unconnected-(U3-PB2-Pad7)")
 			(pinfunction "PB2")
 			(pintype "bidirectional")
@@
 	(footprint "LED_SMD:LED_0805_2012Metric"
 		(layer "F.Cu")
-		(at 97 125.1 -90)
+		(at 97 124.4 -90)
 		(descr "LED SMD 0805 (2012 Metric), square (rectangular) end terminal, IPC-7351 nominal, (Body size source: https://docs.google.com/spreadsheets/d/1BsfQQcO9C6DZCsRaXUlFlo91Tg2WpOkGARC1WS5S8t0/edit?usp=sharing), generated with kicad-footprint-generator")
 		(tags "LED")
 		(property "Reference" "D4"
-			(at 0 -1.65 270)
+			(at -3.1 0.2 180)
 			(layer "F.SilkS")
 			(effects
@@
 		)
 		(property "Value" "LED"
-			(at 0 1.65 270)
+			(at 0 1.65 90)
 			(layer "F.Fab")
+			(hide yes)
 			(effects
 				(font
@@
 		)
 		(property "Datasheet" "~"
-			(at 0 0 270)
+			(at 0 0 90)
 			(layer "F.Fab")
 			(hide yes)
@@
 		)
 		(property "Description" "Light emitting diode"
-			(at 0 0 270)
+			(at 0 0 90)
 			(layer "F.Fab")
 			(hide yes)
@@
 		)
 		(fp_text user "${REFERENCE}"
-			(at 0 0 270)
+			(at 0 0 90)
 			(layer "F.Fab")
 			(effects
@@
 		)
 		(fp_text user "${REFERENCE}"
-			(at 0 -2 270)
+			(at 0.025 0 270)
 			(layer "F.Fab")
 			(effects
@@
 			(layers "*.Cu" "*.Mask")
 			(remove_unused_layers no)
-			(net 12 "Net-(J7-Pin_1)")
+			(net 12 "unconnected-(J7-Pin_1-Pad1)")
 			(pinfunction "Pin_1")
 			(pintype "passive")
@@
 		)
 	)
+	(gr_text "MAXIMUM 30 AMP TOTAL CONSUMPTION!!!"
+		(at 82 122.6 90)
+		(layer "F.SilkS")
+		(effects
+			(font
+				(size 1.2 1.2)
+				(thickness 0.3)
+				(bold yes)
+			)
+			(justify left bottom)
+		)
+	)
 	(gr_text "On-Off-Auto Sw"
 		(at 113.3 107.861252 90)
@@
 		)
 	)
-	(gr_text "Vehicle Power Switch v2.1.1\nZack Clobes, W0ZC\nCustom Digital Services, LLC"
+	(gr_text "Vehicle Power Switch v2.1.2\nZack Clobes, W0ZC\nCustom Digital Services, LLC"
 		(at 90.5 60.9 0)
 		(layer "B.SilkS")
@@
 	)
 	(via
+		(at 101.6 126)
+		(size 0.6)
+		(drill 0.3)
+		(layers "F.Cu" "B.Cu")
+		(free yes)
+		(net 2)
+	)
+	(via
 		(at 76.4 57.1)
 		(size 0.6)
@@
 	)
 	(via
-		(at 99.3 125.1)
+		(at 96 127.2)
 		(size 0.6)
 		(drill 0.3)
@@
 	)
 	(segment
-		(start 101.971 122.669387)
-		(end 101.971 124.776224)
+		(start 109.349 121.151)
+		(end 108.902 121.598)
 		(width 0.2)
 		(layer "F.Cu")
@@
 	)
 	(segment
-		(start 101.971 124.776224)
-		(end 100.247224 126.5)
+		(start 111.225 116.5)
+		(end 110.4 116.5)
 		(width 0.2)
 		(layer "F.Cu")
@@
 	)
 	(segment
-		(start 110.4 116.5)
-		(end 109.349 117.551)
+		(start 97.1375 125.2)
+		(end 97 125.3375)
 		(width 0.2)
 		(layer "F.Cu")
@@
 	)
 	(segment
-		(start 109.349 121.151)
-		(end 108.902 121.598)
+		(start 103.505611 121.598)
+		(end 101.971 123.132612)
 		(width 0.2)
 		(layer "F.Cu")
@@
 	)
 	(segment
-		(start 111.225 116.5)
-		(end 110.4 116.5)
+		(start 101.971 123.132612)
+		(end 99.903611 125.2)
 		(width 0.2)
 		(layer "F.Cu")
@@
 	)
 	(segment
-		(start 108.902 121.598)
-		(end 103.042385 121.598)
+		(start 110.4 116.5)
+		(end 109.349 117.551)
 		(width 0.2)
 		(layer "F.Cu")
@@
 	)
 	(segment
-		(start 100.247224 126.5)
-		(end 97 126.5)
+		(start 99.903611 125.2)
+		(end 97.1375 125.2)
 		(width 0.2)
 		(layer "F.Cu")
@@
 	)
 	(segment
-		(start 103.042385 121.598)
-		(end 101.971 122.669387)
+		(start 108.902 121.598)
+		(end 103.505611 121.598)
 		(width 0.2)
 		(layer "F.Cu")
@@
 	)
 	(segment
-		(start 94 125.3725)
-		(end 95.3275 125.3725)
-		(width 0.2)
-		(layer "F.Cu")
-		(net 10)
-	)
-	(segment
-		(start 95.3275 125.3725)
+		(start 96.35 123.7)
 		(end 97 123.7)
 		(width 0.2)
@@
 	)
 	(segment
-		(start 102.322 124.921612)
-		(end 98.643612 128.6)
+		(start 94 125.3725)
+		(end 94.6775 125.3725)
 		(width 0.2)
 		(layer "F.Cu")
-		(net 11)
+		(net 10)
 	)
 	(segment
-		(start 109.7 121.338612)
-		(end 109.089612 121.949)
+		(start 94.6775 125.3725)
+		(end 96.35 123.7)
 		(width 0.2)
 		(layer "F.Cu")
-		(net 11)
+		(net 10)
 	)
 	(segment
-		(start 103.187775 121.949)
-		(end 102.322 122.814776)
+		(start 94.9 129.7)
+		(end 94.9 130.3)
 		(width 0.2)
 		(layer "F.Cu")
@@
 	)
 	(segment
-		(start 109.089612 121.949)
-		(end 103.187775 121.949)
+		(start 110.66 119.04)
+		(end 109.7 120)
 		(width 0.2)
 		(layer "F.Cu")
@@
 	)
 	(segment
-		(start 102.322 122.814776)
-		(end 102.322 124.921612)
+		(start 97 128.6)
+		(end 96 128.6)
 		(width 0.2)
 		(layer "F.Cu")
@@
 	)
 	(segment
-		(start 110.66 119.04)
-		(end 109.7 120)
+		(start 96 128.6)
+		(end 94.9 129.7)
 		(width 0.2)
 		(layer "F.Cu")
@@
 	)
 	(segment
-		(start 96.707724 128.6)
-		(end 95.007724 130.3)
+		(start 111.225 119.04)
+		(end 110.66 119.04)
 		(width 0.2)
 		(layer "F.Cu")
@@
 	)
 	(segment
-		(start 95.007724 130.3)
-		(end 94.9 130.3)
+		(start 109.089612 121.949)
+		(end 103.651 121.949)
 		(width 0.2)
 		(layer "F.Cu")
@@
 	)
 	(segment
-		(start 98.643612 128.6)
-		(end 96.707724 128.6)
+		(start 103.651 121.949)
+		(end 97 128.6)
 		(width 0.2)
 		(layer "F.Cu")
@@
 	)
 	(segment
-		(start 111.225 119.04)
-		(end 110.66 119.04)
+		(start 109.7 121.338612)
+		(end 109.089612 121.949)
 		(width 0.2)
 		(layer "F.Cu")
@@
 	)
 	(segment
-		(start 102.673 122.960164)
-		(end 102.673 125.067)
-		(width 0.2)
-		(layer "F.Cu")
-		(net 12)
-	)
-	(segment
-		(start 103.333164 122.3)
-		(end 102.673 122.960164)
-		(width 0.2)
-		(layer "F.Cu")
-		(net 12)
-	)
-	(segment
-		(start 102.673 125.067)
-		(end 97.44 130.3)
-		(width 0.2)
-		(layer "F.Cu")
-		(net 12)
-	)
-	(segment
-		(start 111.225 120.31)
-		(end 109.235 122.3)
-		(width 0.2)
-		(layer "F.Cu")
-		(net 12)
-	)
-	(segment
-		(start 109.235 122.3)
-		(end 103.333164 122.3)
-		(width 0.2)
-		(layer "F.Cu")
-		(net 12)
-	)
-	(segment
