File: PCB/Vehicle Power Switch.kicad_sch (KiCad schematic)
At the start: 47 parts, among them J6 STX-3790-5N, J7 Debug Hdr, J8 AVR-UPDI-6, Q1 MMBT2222A, Q2 MMBT2222A, Q3 BSS84, U1 MCP1703Ax-250xxTT, U2 LIS2HH12, U3 ATtiny404-SS

Commit message: Fixes to PCB v2 and working on firmware.
Connections:
- net GND: now also U2.5 (RES)
Changed lines of the file:
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@@
 (kicad_sch
-	(version 20231120)
+	(version 20250114)
 	(generator "eeschema")
-	(generator_version "8.0")
+	(generator_version "9.0")
 	(paper "A4")
 	(junction
@@
 	)
 	(junction
+		(at 144.78 142.24)
+		(diameter 0)
+		(color 0 0 0 0)
+	)
+	(junction
 		(at 241.3 191.77)
 		(diameter 0)
@@
 	(wire
 		(pts
+			(xy 144.78 142.24) (xy 144.78 140.97)
+		)
+		(stroke
+			(width 0)
+			(type default)
+		)
+	)
+	(wire
+		(pts
 			(xy 262.89 93.98) (xy 262.89 99.06)
 		)
@@
 	(wire
 		(pts
+			(xy 144.78 142.24) (xy 132.08 142.24)
+		)
+		(stroke
+			(width 0)
+			(type default)
+		)
+	)
+	(wire
+		(pts
 			(xy 273.05 115.57) (xy 281.94 115.57)
 		)
@@
 	(wire
 		(pts
+			(xy 132.08 142.24) (xy 132.08 135.89)
+		)
+		(stroke
+			(width 0)
+			(type default)
+		)
+	)
+	(wire
+		(pts
 			(xy 59.69 78.74) (xy 69.85 78.74)
 		)
@@
 	(label "1"
 		(at 41.91 130.81 180)
-		(fields_autoplaced yes)
 		(effects
 			(font
@@
 	(label "1"
 		(at 41.91 115.57 180)
-		(fields_autoplaced yes)
 		(effects
 			(font
@@
 	(label "POS"
 		(at 33.02 91.44 180)
-		(fields_autoplaced yes)
 		(effects
 			(font
@@
 	(label "PB1"
 		(at 185.42 125.73 180)
-		(fields_autoplaced yes)
 		(effects
 			(font
@@
 	(label "1"
 		(at 41.91 161.29 180)
-		(fields_autoplaced yes)
 		(effects
 			(font
@@
 	(label "Out3"
 		(at 41.91 146.05 180)
-		(fields_autoplaced yes)
 		(effects
 			(font
@@
 	(label "PB0"
 		(at 185.42 123.19 180)
-		(fields_autoplaced yes)
 		(effects
 			(font
@@
 	(label "POS"
 		(at 33.02 91.44 180)
-		(fields_autoplaced yes)
 		(effects
 			(font
@@
 	(label "Out2"
 		(at 41.91 130.81 180)
-		(fields_autoplaced yes)
 		(effects
 			(font
@@
 	(label "POS"
 		(at 33.02 91.44 180)
-		(fields_autoplaced yes)
 		(effects
 			(font
@@
 	(label "Out1"
 		(at 41.91 115.57 180)
-		(fields_autoplaced yes)
 		(effects
 			(font
@@
 	(label "2"
 		(at 87.63 121.92 180)
-		(fields_autoplaced yes)
 		(effects
 			(font
@@
 	(label "1"
 		(at 41.91 146.05 180)
-		(fields_autoplaced yes)
 		(effects
 			(font
@@
 	(label "Out4"
 		(at 41.91 161.29 180)
-		(fields_autoplaced yes)
 		(effects
 			(font
@@
 	(label "In"
 		(at 33.02 91.44 180)
-		(fields_autoplaced yes)
 		(effects
 			(font
@@
 		(shape input)
 		(at 44.45 90.17 0)
-		(fields_autoplaced yes)
 		(effects
 			(font
@@
 	(symbol
 		(lib_id "power:GND")
-		(at 144.78 140.97 0)
+		(at 144.78 142.24 0)
 		(unit 1)
 		(exclude_from_sim no)
@@
 		(fields_autoplaced yes)
 		(property "Reference" "#PWR013"
-			(at 144.78 147.32 0)
+			(at 144.78 148.59 0)
 			(effects
 				(font
@@
 		)
 		(property "Value" "GND"
-			(at 144.78 146.05 0)
+			(at 144.78 147.32 0)
 			(effects
 				(font
@@
 		)
 		(property "Footprint" ""
-			(at 144.78 140.97 0)
+			(at 144.78 142.24 0)
 			(effects
 				(font
@@
 		)
 		(property "Datasheet" ""
-			(at 144.78 140.97 0)
+			(at 144.78 142.24 0)
 			(effects
 				(font
@@
 		)
 		(property "Description" "Power symbol creates a global label with name \"GND\" , ground"
-			(at 144.78 140.97 0)
+			(at 144.78 142.24 0)
 			(effects
 				(font
@@
 		)
 	)
+	(embedded_fonts no)
 )

Commit message: All functionality is working on the prototype. Firmware is still rough.
Parts:
- added C2: 10nF, Capacitor_SMD:C_0805_2012Metric, symbol Device:C_Polarized_US
- added C3: 22uF, Capacitor_SMD:C_0805_2012Metric, symbol Device:C
- C1: value .1uF -> 22uF; Digikey (none) -> 13-CC0805MFX5R8BB226CT-ND; LCSC (none) -> C16780
- C10: renamed from C9; value .1uF -> 10nF; Digikey (none) -> 399-1158-1-ND; LCSC (none) -> C83170
- C4: renamed from C3; value 10uF -> 10nF; footprint Capacitor_SMD:CP_Elec_4x5.3 -> Capacitor_SMD:C_0805_2012Metric; Digikey (none) -> 399-1158-1-ND; LCSC (none) -> C83170
- C5: renamed from C4; value .1uF -> 10nF; Digikey (none) -> 399-1158-1-ND; LCSC (none) -> C83170
- C6: renamed from C5; value .1uF -> 10nF; Digikey (none) -> 399-1158-1-ND; LCSC (none) -> C83170
- C7: value .1uF -> 10nF; Digikey (none) -> 399-1158-1-ND; LCSC (none) -> C83170
- C8: renamed from C6; value .1uF -> 10nF; Digikey (none) -> 399-1158-1-ND; LCSC (none) -> C83170
- C9: renamed from C8; value .1uF -> 10nF; Digikey (none) -> 399-1158-1-ND; LCSC (none) -> C83170
- D1, D2, D3, D5: value MRA4007T3G -> 1N4007FL; footprint Diode_SMD:D_SMA -> Diode_SMD:D_SOD-123; Digikey (none) -> 1655-1N4007FLCT-ND; LCSC (none) -> C7528871
- D4: footprint LED_SMD:LED_1206_3216Metric -> LED_SMD:LED_0805_2012Metric
- F2, F3, F4, F5: Digikey (none) -> 35-3522-2-ND
- J6: Digikey (none) -> 2092-STX-3790-5N-ND
- K1: renamed from U4; Digikey (none) -> 255-2583-ND
- Q1, Q2: Digikey MMBT2222AFSCT-ND -> 4878-MMBT2222ATR-ND
- U3: Digikey (none) -> ATTINY404-SSFRTR-ND
Connections:
- net +3V3: now also U2.3 (SA0/SDO), C3.1
- net +BATT: now also C2.1
- net GND: now also R7.1, C2.2, C3.2; no longer R7.3
- net at R6.2, U3.13 (PA3): now also R7.3; no longer R7.1
Other:
- moved on the sheet: C1, D1, F1, R7

Commit message: Release candidate for firmware.
Parts:
- F2, F3, F4, F5: Digikey 35-3522-2-ND -> 36-3522-2-ND
Connections:
- net at J7.1 (Pin_1): no longer U3.7 (PB2)
Changed lines of the file:
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@@
 	(wire
 		(pts
-			(xy 182.88 128.27) (xy 182.88 135.89)
-		)
-		(stroke
-			(width 0)
-			(type default)
-		)
-	)
-	(wire
-		(pts
 			(xy 256.54 171.45) (xy 256.54 173.99)
 		)
@@
 	(wire
 		(pts
-			(xy 185.42 128.27) (xy 182.88 128.27)
-		)
-		(stroke
-			(width 0)
-			(type default)
-		)
-	)
-	(wire
-		(pts
 			(xy 72.39 78.74) (xy 87.63 78.74)
 		)
@@
 	(wire
 		(pts
-			(xy 179.07 135.89) (xy 182.88 135.89)
-		)
-		(stroke
-			(width 0)
-			(type default)
-		)
-	)
-	(wire
-		(pts
 			(xy 87.63 121.92) (xy 90.17 121.92)
 		)
@@
 			)
 		)
-		(property "DIGIKEY" ""
-			(at 41.91 115.57 0)
-			(effects
-				(font
-					(size 1.27 1.27)
-				)
-				(hide yes)
-			)
-		)
-		(property "DIGKEY" ""
-			(at 41.91 115.57 0)
-			(effects
-				(font
-					(size 1.27 1.27)
-				)
-				(hide yes)
-			)
-		)
-		(property "Digikey" "35-3522-2-ND"
+		(property "Digikey" "36-3522-2-ND"
 			(at 41.91 115.57 0)
 			(effects
@@
 			)
 		)
-		(property "DIGIKEY" ""
-			(at 41.91 161.29 0)
-			(effects
-				(font
-					(size 1.27 1.27)
-				)
-				(hide yes)
-			)
-		)
-		(property "DIGKEY" ""
-			(at 41.91 161.29 0)
-			(effects
-				(font
-					(size 1.27 1.27)
-				)
-				(hide yes)
-			)
-		)
-		(property "Digikey" "35-3522-2-ND"
+		(property "Digikey" "36-3522-2-ND"
 			(at 41.91 161.29 0)
 			(effects
@@
 			)
 		)
-		(property "DIGIKEY" ""
-			(at 41.91 130.81 0)
-			(effects
-				(font
-					(size 1.27 1.27)
-				)
-				(hide yes)
-			)
-		)
-		(property "DIGKEY" ""
-			(at 41.91 130.81 0)
-			(effects
-				(font
-					(size 1.27 1.27)
-				)
-				(hide yes)
-			)
-		)
-		(property "Digikey" "35-3522-2-ND"
+		(property "Digikey" "36-3522-2-ND"
 			(at 41.91 130.81 0)
 			(effects
@@
 			)
 		)
-		(property "DIGIKEY" ""
-			(at 41.91 146.05 0)
-			(effects
-				(font
-					(size 1.27 1.27)
-				)
-				(hide yes)
-			)
-		)
-		(property "DIGKEY" ""
-			(at 41.91 146.05 0)
-			(effects
-				(font
-					(size 1.27 1.27)
-				)
-				(hide yes)
-			)
-		)
-		(property "Digikey" "35-3522-2-ND"
+		(property "Digikey" "36-3522-2-ND"
 			(at 41.91 146.05 0)
 			(effects
